File: DynOSSAT-EDU-HeaderAdapter.kicad_pcb (KiCad board)
At the start: 4 copper layers, 42 x 42 mm, 11 parts, among them J1 Conn_02x20_Odd_Even, J2 Conn_02x10_Odd_Even, J3 Conn_02x10_Odd_Even

Commit message: Change MISO/MOSI to SDI/SDO
Connections:
- J1 pad 22: /SPI_MOSI -> /SPI_SDO
- J1 pad 26: /SPI_MISO -> /SPI_SDI
Routing:
- net /SPI_SDO: track 0.00 -> 25.3 mm, vias 0 -> 1
- net /SPI_MOSI: track 25.3 -> 0.00 mm, vias 1 -> 0
- net /SPI_SDI: track 0.00 -> 21.8 mm, vias 0 -> 1
- net /SPI_MISO: track 21.8 -> 0.00 mm, vias 1 -> 0
Other:
- board text added: "SDI"
- board text added: "SDO"
- board text removed: "MISO"
- board text removed: "MOSI"
